File: Hardware/Amon_board_STM32H743/power.kicad_sch (KiCad schematic)
At the start: 45 parts, among them J16 XT60PW-M20, J17 XT60PW-M20, J3 Switch_port, U4 MP2303ADN, U5 MP2303ADN

Commit message: Update
compas driver - untested
Parts:
- L1, L2: footprint Inductor_SMD:L_10.4x10.4_H4.8 -> Inductor_SMD:L_APV_APH0630
Changed lines of the file:
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@@
 			)
 		)
-		(property "Footprint" "Inductor_SMD:L_10.4x10.4_H4.8"
+		(property "Footprint" "Inductor_SMD:L_APV_APH0630"
 			(at 149.86 39.37 0)
 			(effects
@@
 			)
 		)
-		(property "Footprint" "Inductor_SMD:L_10.4x10.4_H4.8"
+		(property "Footprint" "Inductor_SMD:L_APV_APH0630"
 			(at 151.13 95.25 0)
 			(effects
