File: Hardware/Amon_board_STM32H743/_autosave-Amon_board.kicad_pcb (KiCad board)
At the start: 4 copper layers, 70 x 120 mm, 142 parts, among them J1 USB2.0_C_Rev, J10 GTFP08131Y2HR, J11 Conn_01x03_Male, J12 Conn_01x06_Male, J13 Conn_01x04_Male, J14 Conn_01x04_Male, J15 Conn_01x06_Male, J16 XT60PW-M20, J17 XT60PW-M20, J3 Switch_port, J4 HAB-VCR-010-LF, J6 Conn_02x04_Odd_Even, J7 Red leds, J8 White leds, J9 Conn_02x04_Odd_Even, M1 Servo_X+, M2 Servo_X-, M3 Servo_Y+, M4 Servo_Y-, Q1 BC817, Q2 BC817, SW1 SW_DPDT, SW2 SW_SPST, U1 USBLC6-2P6, U2 STM32F405RGT6-LQFP64, U3 W25Q128JVS, U4 MP2303ADN, U5 MP2303ADN, U6 MPU-6050, U7 BME280, U8 HMC5883L, U9 STM32H743VIT6, Y1 48MHz, Y2 32.768kHz

Commit message: Update: development of new PCB_v3
Parts:
- removed C1, C2: 15pF, Capacitor_SMD:C_0603_1608Metric
- removed C4, C6: 2.2uF, Capacitor_SMD:C_0603_1608Metric
- removed D1: B120-E3, Diode_SMD:D_SMA
- removed H5, H6: MountingHole, MountingHole:MountingHole_3.2mm_M3
- removed J12: Conn_01x06_Male, Connector_JST:JST_XH_S6B-XH-A-1_1x06_P2.50mm_Horizontal
- removed J6: Conn_02x04_Odd_Even, Connector_PinSocket_2.54mm:PinSocket_2x04_P2.54mm_Vertical
- removed JP3: SolderJumper_2_Open, Jumper:SolderJumper-2_P1.3mm_Open_TrianglePad1.0x1.5mm
- removed R1, R2: 5k1, Resistor_SMD:R_0603_1608Metric
- removed R3: 10k, Resistor_SMD:R_0603_1608Metric
- removed SW1: SW_DPDT, Button_Switch_SMD:SW_SPDT_PCM12
- removed SW2: SW_SPST, Button_Switch_SMD:SW_Push_1P1T_NO_CK_KMR2
- removed U1: USBLC6-2P6, Package_TO_SOT_SMD:SOT-23-6_Handsoldering
- removed U2: STM32F405RGT6-LQFP64, Package_QFP:LQFP-64_10x10mm_P0.5mm
- added C100: 100nF, Capacitor_SMD:C_0603_1608Metric, F.Cu at (104.2, 103.8)
- added C101: 10uF, Capacitor_SMD:C_1206_3216Metric, F.Cu at (115.2, 122.3)
- added C102: 10uF, Capacitor_SMD:C_1206_3216Metric, F.Cu at (98.3, 119.7)
- added C103: 10uF, Capacitor_SMD:C_1206_3216Metric, F.Cu at (80.8, 121.8)
- added C104: 10uF, Capacitor_SMD:C_1206_3216Metric, F.Cu at (80.8, 119.4)
- added C105: 10uF, Capacitor_SMD:C_1206_3216Metric, F.Cu at (80.8, 117.0)
- added C106: 10uF, Capacitor_SMD:C_1206_3216Metric, F.Cu at (98.3, 122.1)
- added C107: 10uF, Capacitor_SMD:C_1206_3216Metric, F.Cu at (98.3, 117.3)
- added C108: 10uF, Capacitor_SMD:C_1206_3216Metric, F.Cu at (115.2, 119.9)
- added C109: 10uF, Capacitor_SMD:C_1206_3216Metric, F.Cu at (115.2, 117.5)
- added C110: 4.7uF, Capacitor_SMD:C_0603_1608Metric, F.Cu at (104.2, 79.5)
- added C111: 4.7uF, Capacitor_SMD:C_0603_1608Metric, F.Cu at (117.2, 92.5)
- added C48: 0.1uF, Capacitor_SMD:C_0603_1608Metric, F.Cu at (121.5, 77.2)
- added C49: 0.1uF, Capacitor_SMD:C_0603_1608Metric, F.Cu at (125.4, 81.9)
- added C50: 10nF, Capacitor_SMD:C_0402_1005Metric, F.Cu at (102.3, 61.2)
- added C51: 10nF, Capacitor_SMD:C_0402_1005Metric, F.Cu at (82.5, 61.2)
- added C52: 33nF, Capacitor_SMD:C_0402_1005Metric, F.Cu at (102.8, 62.9)
- added C53: 33nF, Capacitor_SMD:C_0402_1005Metric, F.Cu at (83.0, 62.9)
- added C54: 1nF, Capacitor_SMD:C_0402_1005Metric, F.Cu at (110.8, 63.0)
- added C55: 1nF, Capacitor_SMD:C_0402_1005Metric, F.Cu at (91.0, 63.0)
- added C56: 1uF, Capacitor_SMD:C_0402_1005Metric, F.Cu at (104.5, 57.8)
- added C57: 1uF, Capacitor_SMD:C_0402_1005Metric, F.Cu at (84.7, 57.8)
- added C58: 22pF, Capacitor_SMD:C_0402_1005Metric, F.Cu at (112.7, 63.0)
- added C59: 22pF, Capacitor_SMD:C_0402_1005Metric, F.Cu at (92.8, 63.0)
- added C60: 22pF, Capacitor_SMD:C_0402_1005Metric, F.Cu at (111.1, 57.8)
- added C61: 22pF, Capacitor_SMD:C_0402_1005Metric, F.Cu at (91.2, 57.7)
- added C62: 2.2nF, Capacitor_SMD:C_0402_1005Metric, F.Cu at (108.4, 55.9)
- added C63: 1.5pF, Capacitor_SMD:C_0402_1005Metric, F.Cu at (106.0, 54.5)
- added C64: 2.2nF, Capacitor_SMD:C_0402_1005Metric, F.Cu at (88.5, 56.8)
- added C65: 1.5pF, Capacitor_SMD:C_0402_1005Metric, F.Cu at (86.0, 54.5)
- added C66: 1pF, Capacitor_SMD:C_0402_1005Metric, F.Cu at (105.5, 53.1)
- added C67: 1pF, Capacitor_SMD:C_0402_1005Metric, F.Cu at (85.5, 53.0)
- added C68: 4.7pF, Capacitor_SMD:C_0402_1005Metric, F.Cu at (108.4, 56.9)
- added C69: 4.7pF, Capacitor_SMD:C_0402_1005Metric, F.Cu at (88.5, 55.8)
- added C70: 220pF, Capacitor_SMD:C_0402_1005Metric, F.Cu at (102.2, 51.2)
- added C71: 220pF, Capacitor_SMD:C_0402_1005Metric, F.Cu at (82.2, 51.2)
- added C72: 0.3pF, Capacitor_SMD:C_0402_1005Metric, F.Cu at (106.0, 47.7)
- added C73: 0.3pF, Capacitor_SMD:C_0402_1005Metric, F.Cu at (86.0, 47.7)
- added C74: 1uF, Capacitor_SMD:C_0402_1005Metric, F.Cu at (102.2, 52.2)
- added C75: 1uF, Capacitor_SMD:C_0402_1005Metric, F.Cu at (82.2, 52.2)
- added C76: 1.5pF, Capacitor_SMD:C_0402_1005Metric, F.Cu at (106.0, 46.7)
- added C77: 1.5pF, Capacitor_SMD:C_0402_1005Metric, F.Cu at (86.0, 46.7)
- added C78: 1.5pF, Capacitor_SMD:C_0402_1005Metric, F.Cu at (106.0, 43.9)
- added C79: 1.5pF, Capacitor_SMD:C_0402_1005Metric, F.Cu at (86.0, 43.9)
- added C80: 1uF, Capacitor_SMD:C_0603_1608Metric, F.Cu at (128.7, 129.2)
- added C81: 1uF, Capacitor_SMD:C_0603_1608Metric, F.Cu at (127.9, 145.2)
- added C82: 0.1uF, Capacitor_SMD:C_0603_1608Metric, F.Cu at (92.1, 107.5)
- added C83: 1uF, Capacitor_SMD:C_0603_1608Metric, F.Cu at (98.3, 106.5)
- added C84: 100nF, Capacitor_SMD:C_0603_1608Metric, F.Cu at (99.3, 105.4)
- added C85: 10nF, Capacitor_SMD:C_0603_1608Metric, F.Cu at (122.0, 71.5)
- added C86: 22pF, Capacitor_SMD:C_0402_1005Metric, F.Cu at (127.4, 70.9)
- added C87: 10uF, Capacitor_Tantalum_SMD:CP_EIA-3216-10_Kemet-I, F.Cu at (122.5, 136.5)
- added C88: 100nF, Capacitor_SMD:C_0603_1608Metric, F.Cu at (112.4, 139.3)
- added C89: 3.9nF, Capacitor_SMD:C_0603_1608Metric, F.Cu at (112.4, 136.2)
- added C90: 10nF, Capacitor_SMD:C_0603_1608Metric, F.Cu at (123.0, 139.6)
- added C91: 22uF, Capacitor_SMD:C_1206_3216Metric, F.Cu at (112.0, 130.0)
- added C92: 22pF, Capacitor_SMD:C_0402_1005Metric, F.Cu at (96.6, 103.3)
- added C93: 22uF, Capacitor_SMD:C_1206_3216Metric, F.Cu at (119.9, 122.3)
- added C94: 22uF, Capacitor_SMD:C_1206_3216Metric, F.Cu at (119.9, 119.9)
- added C95: 100nF, Capacitor_SMD:C_0603_1608Metric, F.Cu at (119.2, 117.5)
- added C96: 100nF, Capacitor_SMD:C_0603_1608Metric, F.Cu at (102.3, 117.3)
- added C97: 100nF, Capacitor_SMD:C_0603_1608Metric, F.Cu at (84.8, 117.0)
- added C98: 100nF, Capacitor_SMD:C_0603_1608Metric, F.Cu at (91.9, 127.1)
- added C99: 100nF, Capacitor_SMD:C_0603_1608Metric, F.Cu at (108.8, 126.9)
- added D10: Red, LED_SMD:LED_0603_1608Metric, F.Cu at (109.3, 134.7)
- added D8: B120-E3, Diode_SMD:D_SMA, F.Cu at (83.4, 110.4)
- added D9: B120-E3, Diode_SMD:D_SMA, F.Cu at (117.6, 132.6)
- added J18: SMA Edge, Connector_Coaxial:SMA_Amphenol_132289_EdgeMount, F.Cu at (105.6, 39.5)
- added J19: SMA Edge, Connector_Coaxial:SMA_Amphenol_132289_EdgeMount, F.Cu at (85.6, 39.5)
- added J2: Conn_01x04_Pin, Connector_JST:JST_EH_S4B-EH_1x04_P2.50mm_Horizontal, F.Cu at (131.0, 137.0)
- added J5: Conn_01x04_Pin, Connector_JST:JST_EH_S4B-EH_1x04_P2.50mm_Horizontal, F.Cu at (131.0, 109.5)
- added L10: 2.4nH, Inductor_SMD:L_0402_1005Metric, F.Cu at (85.5, 45.3)
- added L11: 10uH 4A, Inductor_SMD:L_APV_APH0630, F.Cu at (117.7, 127.1)
- added L3: 8.2nH, Inductor_SMD:L_0402_1005Metric, F.Cu at (106.5, 57.8)
- added L4: 2.7nH, Inductor_SMD:L_0402_1005Metric, F.Cu at (107.0, 56.4)
- added L5: 3.9nH, Inductor_SMD:L_0402_1005Metric, F.Cu at (106.0, 56.4)
- added L6: 8.2nH, Inductor_SMD:L_0402_1005Metric, F.Cu at (86.5, 57.8)
- added L7: 2.7nH, Inductor_SMD:L_0402_1005Metric, F.Cu at (87.0, 56.3)
- added L8: 3.9nH, Inductor_SMD:L_0402_1005Metric, F.Cu at (86.0, 56.3)
- added L9: 2.4nH, Inductor_SMD:L_0402_1005Metric, F.Cu at (105.6, 45.3)
- added Q3: BC817, Package_TO_SOT_SMD:SOT-23, F.Cu at (124.2, 146.6)
- added Q6: BC817, Package_TO_SOT_SMD:SOT-23, F.Cu at (116.7, 141.8)
- added Q7: AO3401A, Package_TO_SOT_SMD:SOT-23, F.Cu at (109.7, 141.8)
- added Q8: BC817, Package_TO_SOT_SMD:SOT-23, F.Cu at (99.6, 141.5)
- added Q9: AO3401A, Package_TO_SOT_SMD:SOT-23, F.Cu at (92.6, 141.5)
- added R42: 22k, Resistor_SMD:R_0402_1005Metric, F.Cu at (102.3, 60.0)
- added R43: 22k, Resistor_SMD:R_0402_1005Metric, F.Cu at (82.5, 60.0)
- added R44: 1M, Resistor_SMD:R_0402_1005Metric, F.Cu at (109.4, 60.4)
- added R45: 1M, Resistor_SMD:R_0402_1005Metric, F.Cu at (89.5, 60.4)
- added R46: 1k, Resistor_SMD:R_0402_1005Metric, F.Cu at (108.6, 51.7)
- added R47: 1k, Resistor_SMD:R_0402_1005Metric, F.Cu at (88.5, 51.6)
- added R48: 1k, Resistor_SMD:R_0402_1005Metric, F.Cu at (108.6, 50.7)
- added R49: 20k, Resistor_SMD:R_0402_1005Metric, F.Cu at (108.6, 49.6)
- added R50: 1k, Resistor_SMD:R_0402_1005Metric, F.Cu at (88.5, 50.6)
- added R51: 20k, Resistor_SMD:R_0402_1005Metric, F.Cu at (88.5, 49.6)
- added R52: 10k, Resistor_SMD:R_0603_1608Metric, F.Cu at (93.8, 86.4)
- added R53: 5k1, Resistor_SMD:R_0603_1608Metric, F.Cu at (129.2, 63.2)
- added R54: 100k, Resistor_SMD:R_0603_1608Metric, F.Cu at (112.4, 137.8)
- added R55: 6k8, Resistor_SMD:R_0603_1608Metric, F.Cu at (109.3, 136.2)
- added R56: 10k, Resistor_SMD:R_0603_1608Metric, F.Cu at (112.4, 134.7)
- added R57: 68k, Resistor_SMD:R_0603_1608Metric, F.Cu at (112.4, 133.1)
- added R58: 1k5, Resistor_SMD:R_0603_1608Metric, F.Cu at (109.3, 133.1)
- added R59: 1k, Resistor_SMD:R_0603_1608Metric, F.Cu at (120.7, 145.7)
- added R60: 1k, Resistor_SMD:R_0603_1608Metric, F.Cu at (120.6, 147.6)
- added R63: 10k, Resistor_SMD:R_0603_1608Metric, F.Cu at (120.3, 141.1)
- added R64: 1k, Resistor_SMD:R_0603_1608Metric, F.Cu at (120.3, 142.8)
- added R65: 10k, Resistor_SMD:R_0603_1608Metric, F.Cu at (113.3, 142.8)
- added R66: 1k, Resistor_SMD:R_0603_1608Metric, F.Cu at (113.2, 141.1)
- added R67: 10k, Resistor_SMD:R_0603_1608Metric, F.Cu at (103.1, 140.8)
- added R68: 1k, Resistor_SMD:R_0603_1608Metric, F.Cu at (103.1, 142.5)
- added R69: 10k, Resistor_SMD:R_0603_1608Metric, F.Cu at (96.1, 142.5)
- added R70: 1k, Resistor_SMD:R_0603_1608Metric, F.Cu at (96.1, 140.8)
- added R71: 10k, Resistor_SMD:R_0603_1608Metric, F.Cu at (92.2, 137.4)
- added R72: 10k, Resistor_SMD:R_0603_1608Metric, F.Cu at (109.3, 137.8)
- added R73: 0R, Resistor_SMD:R_0603_1608Metric, F.Cu at (92.1, 139.0)
- added R74: 0R, Resistor_SMD:R_0603_1608Metric, F.Cu at (109.3, 139.3)
- added R75: 100k, Resistor_SMD:R_0603_1608Metric, F.Cu at (109.3, 131.6)
- added R76: 75k, Resistor_SMD:R_0603_1608Metric, F.Cu at (109.3, 130.0)
- added R77: 100k, Resistor_SMD:R_0603_1608Metric, F.Cu at (92.2, 131.3)
- added R78: 150k, Resistor_SMD:R_0603_1608Metric, F.Cu at (92.2, 129.8)
- added REF**: KiCad-Logo2_5mm_SilkScreen, Symbol:KiCad-Logo2_5mm_SilkScreen, F.Cu at (75.2, 55.5)
- added REF**: OSHW-Logo_7.5x8mm_SilkScreen, Symbol:OSHW-Logo_7.5x8mm_SilkScreen, F.Cu at (91.8, 119.3)
- added SW3: SW_SPST, Button_Switch_SMD:SW_Push_1P1T_NO_CK_KMR2, F.Cu at (89.6, 104.9)
- added U10: NRF24L01, Package_DFN_QFN:QFN-20-1EP_4x4mm_P0.5mm_EP2.5x2.5mm, F.Cu at (106.0, 61.1)
- added U11: NRF24L01, Package_DFN_QFN:QFN-20-1EP_4x4mm_P0.5mm_EP2.5x2.5mm, F.Cu at (86.1, 61.1)
- added U12: RFX2401C, RFX2401C:QFN50P300X300X60-17N, F.Cu at (105.3, 50.4)
- added U13: RFX2401C, RFX2401C:QFN50P300X300X60-17N, F.Cu at (85.2, 50.4)
- added U14: CH340G, Package_SO:SOIC-16_3.9x9.9mm_P1.27mm, F.Cu at (122.7, 66.0)
- added U15: MP2303ADN, Package_SO:SOIC-8-1EP_3.9x4.9mm_P1.27mm_EP2.62x3.51mm, F.Cu at (117.7, 137.1)
- added Y3: 16MHz, Crystal:Crystal_SMD_3225-4Pin_3.2x2.5mm, F.Cu at (111.9, 60.4)
- added Y4: 16MHz, Crystal:Crystal_SMD_3225-4Pin_3.2x2.5mm, F.Cu at (92.0, 60.3)
- added Y5: 12MHz, Crystal:Resonator_SMD_Murata_CSTxExxV-3Pin_3.0x1.1mm, F.Cu at (126.5, 72.7)
- C26: value 10uF -> 10nF; footprint Capacitor_SMD:CP_Elec_4x5.4 -> Capacitor_SMD:C_0603_1608Metric
- C30, C43: value 10uF -> 22pF; footprint Capacitor_SMD:CP_Elec_4x5.4 -> Capacitor_SMD:C_0402_1005Metric
- C42: value 10uF -> 100nF; footprint Capacitor_SMD:CP_Elec_4x5.4 -> Capacitor_SMD:C_0603_1608Metric
- J1: value USB2.0_C_Rev -> USB_C_Receptacle_USB2.0
- J3: value Switch_port -> Conn_01x04_Pin; footprint TerminalBlock_MetzConnect:TerminalBlock_MetzConnect_Type055_RT01502HDWU_1x02_P5.00mm_Horizontal -> Connector_JST:JST_EH_S4B-EH_1x04_P2.50mm_Horizontal
- J7, J8: footprint TerminalBlock_MetzConnect:TerminalBlock_MetzConnect_Type055_RT01502HDWU_1x02_P5.00mm_Horizontal -> TerminalBlock_MetzConnect:TerminalBlock_MetzConnect_Type059_RT06302HBWC_1x02_P3.50mm_Horizontal
- J9: value Conn_02x04_Odd_Even -> AUX; footprint Connector_PinSocket_2.54mm:PinSocket_2x04_P2.54mm_Vertical -> TerminalBlock_MetzConnect:TerminalBlock_MetzConnect_Type059_RT06302HBWC_1x02_P3.50mm_Horizontal
- JP1: footprint Jumper:SolderJumper-2_P1.3mm_Open_Pad1.0x1.5mm -> Jumper:SolderJumper-2_P1.3mm_Open_RoundedPad1.0x1.5mm
- L1, L2: footprint Inductor_SMD:L_10.4x10.4_H4.8 -> Inductor_SMD:L_APV_APH0630
- R36: value 22 -> 10k
- R37: value 22 -> 5k1
- moved C14 139.2 mm to (74.3, 78.6), turned to 180 degrees
- moved R9 136.7 mm to (77.3, 78.6)
- moved C33 132.1 mm to (91.7, 85.3), turned to -135 degrees
- moved U3 131.8 mm to (91.3, 80.5), turned to -135 degrees
- moved R8 131.5 mm to (81.6, 77.1), turned to 0 degrees
- moved R7 131.1 mm to (81.6, 75.5), turned to 0 degrees
- moved R6 130.7 mm to (81.6, 74.0), turned to 0 degrees
- moved R39 121.5 mm to (96.1, 80.8), turned to 45 degrees
- moved C19 120.6 mm to (77.5, 129.7), turned to -90 degrees
- moved R18 115.4 mm to (74.9, 132.8), turned to 180 degrees
- moved L1 114.2 mm to (83.2, 126.7), turned to 180 degrees
- moved D3 114.1 mm to (74.9, 134.3), turned to 180 degrees
- moved R14 112.8 mm to (74.9, 135.8), turned to 0 degrees
- moved R17 112.1 mm to (77.9, 132.8), turned to 180 degrees
- moved R16 110.8 mm to (77.9, 134.3), turned to 0 degrees
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Connections:
- net BAT_BRD_S renamed /Power/AN_BAT_BRD
- net BAT_EDF_S renamed /Power/AN_BAT_EDF
- net CS_SD renamed /Devices/CS_SD
- C26 pad 1: +3V3 -> GND
- C26 pad 2: GND -> Net-(J1-SHIELD)
- C30 pad 1: +3V3 -> GND
- C30 pad 2: GND -> Net-(U14-XI)
- C37 pad 1: VBUS -> GND
- C37 pad 2: GND -> VBUS
- C42 pad 1: +5V -> GND
- C42 pad 2: GND -> +3V3
- C43 pad 1: +3V3 -> /Microcontroller/HSE_IN
- J1 pad A6: Net-(J1-D+-PadA6) -> /Microcontroller/D+
- J1 pad A7: Net-(J1-D--PadA7) -> /Microcontroller/D-
- J1 pad B6: Net-(J1-D+-PadA6) -> /Microcontroller/D+
- J1 pad B7: Net-(J1-D--PadA7) -> /Microcontroller/D-
- J1 pad S1: unconnected-(J1-SHIELD-PadS1) -> Net-(J1-SHIELD)
- J10 pad 3: MOSI -> /Devices/MOSI
- J10 pad 5: CLK -> /Devices/CLK
- J10 pad 7: MISO -> /Devices/MISO
- J11 pad 1: PWM_EDF -> /Outputs/PWM_EDF
- J11 pad 2: +5V -> Net-(J11-Pin_2)
- J13 pad 2: TX_GPS -> /Outputs/TX_GPS
- J13 pad 3: RX_GPS -> /Outputs/RX_GPS
- J14 pad 2: SDA -> /Outputs/SDA_EXT
- J14 pad 3: SCL -> /Outputs/SCL_EXT
- J15 pad 2: MISO -> /Outputs/MISO_EXT
- J15 pad 3: CLK -> /Outputs/CLK_EXT
- J15 pad 4: MOSI -> /Outputs/MOSI_EXT
- J15 pad 5: CS_EXT -> /Outputs/CS_EXT
- J16 pad 2: /Power/VBAT+ -> Net-(D8-A)
- J3 pad 1: Net-(D1-A) -> /Outputs/CLK
- J3 pad 2: /Power/VBAT+ -> /Outputs/MOSI
- J9 pad 1: +3V3 -> Net-(J9-Pin_1)
- JP1 pad 1: Net-(D1-A) -> Net-(J11-Pin_2)
- JP1 pad 2: /Power/VBAT+ -> +5V
- M1 pad 1: PWM_Servo_X+ -> /Outputs/PWM_Servo_X+
- M1 pad 2: +5V -> +7V2
- M2 pad 1: PWM_Servo_X- -> /Outputs/PWM_Servo_X-
- M2 pad 2: +5V -> +7V2
- M3 pad 1: PWM_Servo_Y+ -> /Outputs/PWM_Servo_Y+
- M3 pad 2: +5V -> +7V2
- M4 pad 1: PWM_Servo_Y- -> /Outputs/PWM_Servo_Y-
- M4 pad 2: +5V -> +7V2
- R19 pad 1: /Power/12V -> Net-(Q9-D)
- R24 pad 2: LED_Red -> /Outputs/LED_Red
- R25 pad 2: LED_White -> /Outputs/LED_White
- R29 pad 2: MISO -> /Devices/MISO
- R30 pad 2: CLK -> /Devices/CLK
- R31 pad 2: MOSI -> /Devices/MOSI
- R32 pad 1: Brd_Led -> /Devices/BRD_Led
- R33 pad 1: RGB_Led_R -> /Devices/RGB_Led_R
- R34 pad 1: RGB_Led_G -> /Devices/RGB_Led_G
- R35 pad 1: RGB_Led_B -> /Devices/RGB_Led_B
- R36 pad 1: Net-(J1-D--PadA7) -> GND
- R36 pad 2: /IN_D- -> Net-(J1-SHIELD)
- R37 pad 1: Net-(J1-D+-PadA6) -> GND
- R37 pad 2: /IN_D+ -> Net-(J1-CC1)
- R39 pad 2: CS_Flash -> /Microcontroller/CS_F
- U3 pad 1: CS_Flash -> /Microcontroller/CS_F
- U3 pad 2: MISO -> /Microcontroller/MISO_F
- U3 pad 5: MOSI -> /Microcontroller/MOSI_F
- U3 pad 6: CLK -> /Microcontroller/SCK_F
- U6 pad 23: SCL -> /Devices/SCL
- U6 pad 24: SDA -> /Devices/SDA
- U7 pad 3: SDA -> /Devices/SDA
- U7 pad 4: SCL -> /Devices/SCL
- U8 pad 1: SCL -> /Devices/SCL
- U8 pad 15: unconnected-(U8-DRDY-Pad15) -> /Devices/DRDY
- U8 pad 16: SDA -> /Devices/SDA
- U9 pad 1: unconnected-(U9-PE2-Pad1) -> /Microcontroller/SCK_F
- U9 pad 100: unconnected-(U9-VDD-Pad100) -> +3V3
- U9 pad 11: unconnected-(U9-VDD-Pad11) -> +3V3
- U9 pad 12: unconnected-(U9-PH0-Pad12) -> /Microcontroller/HSE_IN
- U9 pad 13: unconnected-(U9-PH1-Pad13) -> /Microcontroller/HSE_OUT
- U9 pad 14: unconnected-(U9-NRST-Pad14) -> /Microcontroller/NRST
- U9 pad 2: unconnected-(U9-PE3-Pad2) -> /Microcontroller/CS_F
- U9 pad 20: unconnected-(U9-VREF+-Pad20) -> +3V3
- U9 pad 21: unconnected-(U9-VDDA-Pad21) -> +3.3VA
- U9 pad 27: unconnected-(U9-VDD-Pad27) -> +3V3
- U9 pad 4: unconnected-(U9-PE5-Pad4) -> /Microcontroller/MISO_F
- U9 pad 48: unconnected-(U9-VCAP-Pad48) -> Net-(C111-Pad1)
- U9 pad 5: unconnected-(U9-PE6-Pad5) -> /Microcontroller/MOSI_F
- U9 pad 50: unconnected-(U9-VDD-Pad50) -> +3V3
- U9 pad 6: unconnected-(U9-VBAT-Pad6) -> +3V3
- U9 pad 72: unconnected-(U9-PA13-Pad72) -> /Microcontroller/SWDIO
- U9 pad 73: unconnected-(U9-VCAP-Pad73) -> Net-(C110-Pad1)
- U9 pad 75: unconnected-(U9-VDD-Pad75) -> +3V3
- U9 pad 76: unconnected-(U9-PA14-Pad76) -> /Microcontroller/SWDCLK
- U9 pad 8: unconnected-(U9-PC14-Pad8) -> /Microcontroller/LSE_IN
- U9 pad 89: unconnected-(U9-PB3-Pad89) -> /Microcontroller/SWO
- U9 pad 9: unconnected-(U9-PC15-Pad9) -> /Microcontroller/LSE_OUT
- U9 pad 94: unconnected-(U9-BOOT0-Pad94) -> Net-(U9-BOOT0)
Routing:
- net MOSI: track 122.3 -> 0.00 mm, vias 3 -> 0
- net CLK: track 119.5 -> 0.00 mm, vias 3 -> 0
- net SCL: track 98.6 -> 0.00 mm, vias 2 -> 0
- net SDA: track 96.7 -> 0.00 mm, vias 1 -> 0
- net MISO: track 96.2 -> 0.00 mm, vias 2 -> 0
- net GND: track 18.5 -> 96.1 mm, vias 63 -> 200
- net /NRST: track 71.8 -> 0.00 mm, vias 2 -> 0
- net PWM_Servo_X+: track 62.6 -> 0.00 mm, vias 1 -> 0
- net PWM_Servo_X-: track 60.3 -> 0.00 mm, vias 1 -> 0
- net /Power/12V: track 89.9 -> 35.8 mm
- net PWM_EDF: track 53.6 -> 0.00 mm, vias 1 -> 0
- net TX_GPS: track 53.2 -> 0.00 mm
- net LED_White: track 53.0 -> 0.00 mm, vias 2 -> 0
- net PWM_Servo_Y-: track 52.8 -> 0.00 mm, vias 1 -> 0
- net RX_GPS: track 52.3 -> 0.00 mm
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- added copper zone on F.Cu, net +7V2
- added copper zone on In2.Cu, net +7V2
- added copper zone on F.Cu, net /Power/12V
- added copper zone on F.Cu, net Net-(D8-A)
- added copper zone on F.Cu, net Net-(D9-K)
- added copper zone on F.Cu, net Net-(J1-SHIELD)
- removed copper zone on F.Cu, net /Power/VBAT+
- removed copper zone on F.Cu, net Net-(D1-A)
Other:
- board text added: "AUX"
- board text added: "ESC PWR"
- board text added: "MAIN"
- board text added: "O. FLOW"
- board text added: "R1"
- board text added: "R2"
- board text added: "Rev.: 3.0, May 2026"
- board text added: "TOF"
- board text removed: "CS1"
- board text removed: "CS2"
- board text removed: "EN1"
- board text removed: "EN2"
- board text removed: "IRQ1"
- board text removed: "IRQ2"
- board text removed: "LIDAR"
- board text removed: "NC"
- board text removed: "ON/OFF"
- board text removed: "PWR"
- board text removed: "RADIO 1"
- board text removed: "RADIO 2"
- board text removed: "RST"
- board text removed: "RUN|BOOT"
- board text removed: "Rev.: 2.2, February 2023"
- board text removed: "SWDIO"
- board text removed: "SWO"
- board text removed: "Sense - EDF"
