File: Hardware/Amon_board_STM32H743/_autosave-microcontroller.kicad_sch (KiCad schematic)
At the start: 51 parts, among them J1 USB_C_Receptacle_USB2.0, J4 HAB-VCR-010-LF, SW3 SW_SPST, U14 CH340G, U3 W25Q128JVS, U9 STM32H743VIT6, Y1 48MHz, Y2 32.768kHz, Y5 12MHz

Commit message: Update: finished routing of PCB_v3
Parts:
- removed R38, R40, R41: 10k, Resistor_SMD:R_0603_1608Metric, symbol Device:R
- removed R4, R5: 4k7, Resistor_SMD:R_0603_1608Metric, symbol Device:R_Small
- added R38, R85: 0R, Resistor_SMD:R_0603_1608Metric, symbol Device:R_Small
- added R40, R41, R81, R84: 4k7, Resistor_SMD:R_0603_1608Metric, symbol Device:R_Small
Connections:
- net +3V3: now also R40.1, R41.1, R81.1, R84.1
- net AN_BUCK_7V2: now also U9.30 (PA6)
- net CS_EXT: now also U9.37 (PE7)
- net CS_SD: now also U9.44 (PE14)
- net LED_Red: now also U9.32 (PC4)
- net LED_White: now also U9.33 (PC5)
- net PWM_EDF: now also U9.35 (PB1)
- net PWM_Servo_X+: now also U9.22 (PA0)
- net PWM_Servo_X-: now also U9.23 (PA1)
- net PWM_Servo_Y+: now also U9.24 (PA2)
- net PWM_Servo_Y-: now also U9.25 (PA3)
- net RGB_Led_B: now also U9.95 (PB8)
- net RGB_Led_G: now also U9.93 (PB7)
- net RGB_Led_R: now also U9.92 (PB6)
- net RXD: now also U9.51 (PB12), R85.1; no longer U14.3 (RXD)
- net RX_GPS: now also U9.53 (PB14)
- net TXD: now also U9.52 (PB13), R38.1; no longer U14.2 (TXD)
- net TX_GPS: now also U9.54 (PB15)
- net AN_BAT_EDF: now reaches U9.15 (PC0)
- net AN_BAT_MAIN: now reaches U9.16 (PC1)
- net MISO_S: now reaches U9.17 (PC2_C)
- net MOSI_S: now reaches U9.18 (PC3_C)
- net AN_BUCK_5V: now reaches U9.28 (PA4)
- net BUCK_EN_5V: now reaches U9.29 (PA5)
- net BUCK_EN_7V2: now reaches U9.31 (PA7)
- net AUX_port: now reaches U9.34 (PB0)
- net CS_OF: now reaches U9.41 (PE11)
- net RST: now reaches U9.42 (PE12)
- net MOT: now reaches U9.43 (PE13)
- net DRDY: now reaches U9.45 (PE15)
- net SCL_S: now reaches U9.46 (PB10)
- net SCL_S: now also R40.2
- net SDA_S: now reaches U9.47 (PB11)
- net SDA_S: now also R41.2
- net SCL_EXT: now reaches U9.59 (PD12)
- net SCL_EXT: now also R81.2
- net SDA_EXT: now reaches U9.60 (PD13)
- net SDA_EXT: now also R84.2
- net CLK_S: now reaches U9.68 (PA9)
- net IRQ1: now reaches U9.71 (PA12)
- net SCK_RF: now reaches U9.78 (PC10)
- net MISO_RF: now reaches U9.79 (PC11)
- net MOSI_RF: now reaches U9.80 (PC12)
- net CSN1: now reaches U9.81 (PD0)
- net CE1: now reaches U9.82 (PD1)
- net IRQ2: now reaches U9.86 (PD5)
- net CSN2: now reaches U9.87 (PD6)
- net CE2: now reaches U9.88 (PD7)
- net BRD_Led: now reaches U9.96 (PB9)
- net SWDCLK renamed SWCLK
- new net: R38.2, U14.2 (TXD)
- new net: R85.2, U14.3 (RXD)
- no-connect marks 18 -> 38
Other:
- note removed: "make PWR copper pour on pins"
- moved on the sheet: C110, C111, C14, C30, C37, C42, C82, C85, C86, J4, R52, R6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
