File: Hardware/Amon_board_STM32H743/_autosave-outputs.kicad_sch (KiCad schematic)
At the start: 26 parts, among them J11 Conn_01x03_Male, J13 Conn_01x04_Male, J14 Conn_01x04_Male, J15 Conn_01x06_Male, J2 Conn_01x04_Pin, J3 Conn_01x04_Pin, J5 Conn_01x04_Pin, J7 Red leds, J8 White leds, J9 AUX, M1 Servo_X+, M2 Servo_X-, M3 Servo_Y+, M4 Servo_Y-, Q1 BC817, Q2 BC817, Q3 BC817

Commit message: Update: finished routing of PCB_v3
Parts:
- removed C80, C81: 1uF, Capacitor_SMD:C_0603_1608Metric, symbol Device:C_Small
- removed J2, J3, J5: Conn_01x04_Pin, Connector_JST:JST_EH_S4B-EH_1x04_P2.50mm_Horizontal, symbol Connector:Conn_01x04_Pin
- added R82: 10k, Resistor_SMD:R_0603_1608Metric, symbol Device:R_Small
Connections:
- net +3V3: now also R82.2
- net CS_EXT: now also R82.1
- net RX_GPS: now also J13.2 (Pin_2); no longer J13.3 (Pin_3)
- net TX_GPS: now also J13.3 (Pin_3); no longer J13.2 (Pin_2)
- net CLK_EXT renamed CLK_S
- net MISO_EXT renamed MISO_S
- net MOSI_EXT renamed MOSI_S
Other:
- note removed: "OPTICAL FLOW:"
- note removed: "PMW3901"
- note removed: "TOF400C-VL53L1X"
- note removed: "TOF:"
- moved on the sheet: J15
