File: Hardware/Amon_board_STM32H743/_autosave-power.kicad_sch (KiCad schematic)
At the start: 91 parts, among them J16 XT60PW-M20, J17 XT60PW-M20, Q6 BC817, Q7 AO3401A, Q8 BC817, Q9 AO3401A, U15 MP2303ADN, U4 MP2303ADN, U5 MP2303ADN

Commit message: Update: finished routing of PCB_v3
Connections:
- net AN_BAT_BRD renamed AN_BAT_MAIN
Changed lines of the file:
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@@
 		)
 	)
-	(hierarchical_label "AN_BAT_BRD"
+	(hierarchical_label "AN_BAT_MAIN"
 		(shape output)
 		(at 259.08 62.23 0)
