File: Hardware/Amon_board_STM32H743/_autosave-rf.kicad_sch (KiCad schematic)
At the start: 56 parts, among them J18 SMA Edge, J19 SMA Edge, U10 NRF24L01, U11 NRF24L01, U12 RFX2401C, U13 RFX2401C, Y3 16MHz, Y4 16MHz

Commit message: Update: finished routing of PCB_v3
Parts:
- added R61, R62: 10k, Resistor_SMD:R_0603_1608Metric, symbol Device:R
Connections:
- net +3V3: now also R61.1, R62.1
- net CSN1: now also R61.2
- net CSN2: now also R62.2
