File: Hardware/Amon_board_STM32H743/_autosave-sensors.kicad_sch (KiCad schematic)
At the start: 26 parts, among them J10 GTFP08131Y2HR, U6 MPU-6050, U7 BME280, U8 HMC5883L

Commit message: Update: finished routing of PCB_v3
Parts:
- added C80, C81: 1uF, Capacitor_SMD:C_0603_1608Metric, symbol Device:C_Small
- added J2, J3, J5: Conn_01x04_Pin, Connector_JST:JST_EH_S4B-EH_1x04_P2.50mm_Horizontal, symbol Connector:Conn_01x04_Pin
- added R83: 10k, Resistor_SMD:R_0603_1608Metric, symbol Device:R_Small
Connections:
- net +3V3: now also C80.1, C81.1, J2.4 (Pin_4), J3.4 (Pin_4), R83.2
- net GND: now also C80.2, C81.2, J2.3 (Pin_3), J3.3 (Pin_3)
- net CLK renamed CLK_S
- net CLK_S: now also J3.1 (Pin_1)
- net MISO renamed MISO_S
- net MISO_S: now also J5.4 (Pin_4)
- net MOSI renamed MOSI_S
- net MOSI_S: now also J3.2 (Pin_2)
- net SCL renamed SCL_S
- net SCL_S: now also J2.2 (Pin_2)
- net SDA renamed SDA_S
- net SDA_S: now also J2.1 (Pin_1)
- new net CS_OF: J5.3 (Pin_3), R83.1
- new net MOT: J5.1 (Pin_1)
- new net RST: J5.2 (Pin_2)
Other:
- note added: "OPTICAL FLOW:"
- note added: "PMW3901"
- note added: "TOF400C-VL53L1X"
- note added: "TOF:"
