File: Hardware/Amon_board_STM32H743/sensors.kicad_sch (KiCad schematic)
At the start: 32 parts, among them J10 GTFP08131Y2HR, J2 Conn_01x04_Pin, J3 Conn_01x04_Pin, J5 Conn_01x04_Pin, U6 MPU-6050, U7 BME280, U8 HMC5883L

Commit message: Update: NMPC development, 1st order model, single file selection
Other:
- title: Amon board - Sensors -> Amon board - Devices
Changed lines of the file:
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@@
 	(paper "A4")
 	(title_block
-		(title "Amon board - Sensors")
+		(title "Amon board - Devices")
 		(date "2026-05-10")
 		(rev "3.0")
